Commit message: modified : xacro description of robaato.

File: robaato_description/urdf/macros.xacro (robot description, xacro)
@@ -31,6 +31,6 @@
     />
   </xacro:macro>
-  <xacro:macro name="tof_sensor" params="tof_number pos_x pos_y pos_z ang_r ang_p ang_y">
-    <link name="tof_${tof_number}_link">
+  <xacro:macro name="tof_sensor" params="tof_name pos_x pos_y pos_z ang_r ang_p ang_y">
+    <link name="tof_${tof_name}_link">
       <inertial>
         <origin xyz="${-tof_x/2} 0 ${tof_z/2-tof_h}" rpy="0 0 0"/>
@@ -57,11 +57,11 @@
       </collision>
     </link>
-    <joint name="tof_${tof_number}_joint" type="fixed">
+    <joint name="tof_${tof_name}_joint" type="fixed">
       <origin xyz="${pos_x+tof_x/2} ${pos_y} ${pos_z+chassis_z/2+tof_h}" rpy="${ang_r} ${ang_p} ${ang_y}"/>
       <parent link="chassis"/>
-      <child link="tof_${tof_number}_link"/>
+      <child link="tof_${tof_name}_link"/>
     </joint>
-    <gazebo reference="tof_${tof_number}_link">
-      <sensor type="ray" name="tof_${tof_number}">
+    <gazebo reference="tof_${tof_name}_link">
+      <sensor type="ray" name="tof_${tof_name}">
         <pose>0 0 0 0 0 0</pose>
         <ray>
@@ -81,6 +81,6 @@
         </ray>
         <plugin name="laser" filename="libgazebo_ros_laser.so">
-          <topicName>tof_${tof_number}/scan</topicName>
-          <frameName>tof_${tof_number}_link</frameName>
+          <topicName>tof_${tof_name}/scan</topicName>
+          <frameName>tof_${tof_name}_link</frameName>
         </plugin>
         <alwaysOn>1</alwaysOn>

File: robaato_description/urdf/robaato.xacro (robot description, xacro)
@@ -5,4 +5,14 @@
   <xacro:include filename="$(find robaato_description)/urdf/macros.xacro"/>
   <xacro:include filename="$(find robaato_description)/urdf/properties.xacro"/>
+  <link name="base_link">
+    <inertial>
+      <origin xyz="0 0 0" rpy="0 0 0"/>
+      <mass value="0.0"/>
+      <xacro:sphere_inertia
+        m="0.0"
+        r="0.1"
+      />
+    </inertial>
+  </link>
   <link name="chassis">
     <inertial>
@@ -91,4 +101,9 @@
     </collision>
   </link>
+  <joint name="chassis_joint" type="fixed">
+    <origin xyz="${chassis_x/2-wheel_dx} 0 ${chassis_z/2-wheel_dz}" rpy="0 0 0"/>
+    <parent link="base_link"/>
+    <child link="chassis"/>
+  </joint>
   <joint name="left_wheel_joint" type="continuous">
     <origin xyz="${-chassis_x/2+wheel_dx} ${chassis_y/2+wheel_dy+wheel_d/2} ${-chassis_z/2+wheel_dz}" rpy="0 0 0"/>
@@ -107,5 +122,5 @@
   </joint>
   <xacro:tof_sensor
-    tof_number="a"
+    tof_name="fm"
     pos_x="${chassis_x*0.4}"
     pos_y="0"
@@ -116,5 +131,5 @@
   />
   <xacro:tof_sensor
-    tof_number="b"
+    tof_name="fl"
     pos_x="${chassis_x*0.35}"
     pos_y="${chassis_y*0.35}"
@@ -125,5 +140,5 @@
   />
   <xacro:tof_sensor
-    tof_number="c"
+    tof_name="fr"
     pos_x="${chassis_x*0.35}"
     pos_y="${-chassis_y*0.35}"
@@ -134,5 +149,5 @@
   />
   <xacro:tof_sensor
-    tof_number="d"
+    tof_name="sl"
     pos_x="${-chassis_x*0.2}"
     pos_y="${chassis_y*0.35}"
@@ -143,5 +158,5 @@
   />
   <xacro:tof_sensor
-    tof_number="e"
+    tof_name="sr"
     pos_x="${-chassis_x*0.2}"
     pos_y="${-chassis_y*0.35}"
@@ -152,5 +167,5 @@
   />
   <xacro:tof_sensor
-    tof_number="f"
+    tof_name="bm"
     pos_x="${-chassis_x*0.4}"
     pos_y="0"
