Commit message: modified : Achieved blind odometry.

File: robaato_description/urdf/properties.xacro (robot description, xacro)
@@ -5,8 +5,8 @@
   <xacro:property name="chassis_y" value="0.31400"/>
   <xacro:property name="chassis_z" value="0.11900"/>
-  <xacro:property name="chassis_w" value="1.00000"/>
+  <xacro:property name="chassis_w" value="3.00000"/>
   <xacro:property name="wheel_r" value="0.0350"/>
   <xacro:property name="wheel_d" value="0.0240"/>
-  <xacro:property name="wheel_w" value="0.2000"/>
+  <xacro:property name="wheel_w" value="0.1000"/>
   <xacro:property name="wheel_dx" value="0.04848"/>
   <xacro:property name="wheel_dy" value="0.00850"/>

File: robaato_description/urdf/robaato.xacro (robot description, xacro)
@@ -123,5 +123,5 @@
   <xacro:tof_sensor
     tof_name="fm"
-    pos_x="${chassis_x*0.4}"
+    pos_x="${0.1675}"
     pos_y="0"
     pos_z="0"
@@ -132,41 +132,41 @@
   <xacro:tof_sensor
     tof_name="fl"
-    pos_x="${chassis_x*0.35}"
-    pos_y="${chassis_y*0.35}"
+    pos_x="${0.11698}"
+    pos_y="${0.12504}"
     pos_z="0"
     ang_r="0"
     ang_p="0"
-    ang_y="${PI/6}"
+    ang_y="${44*PI/180}"
   />
   <xacro:tof_sensor
     tof_name="fr"
-    pos_x="${chassis_x*0.35}"
-    pos_y="${-chassis_y*0.35}"
+    pos_x="${0.11698}"
+    pos_y="${-0.12504}"
     pos_z="0"
     ang_r="0"
     ang_p="0"
-    ang_y="${-PI/6}"
+    ang_y="${-44*PI/180}"
   />
   <xacro:tof_sensor
     tof_name="sl"
-    pos_x="${-chassis_x*0.2}"
-    pos_y="${chassis_y*0.35}"
+    pos_x="${-0.0125}"
+    pos_y="${0.145}"
     pos_z="0"
     ang_r="0"
     ang_p="0"
-    ang_y="${2*PI/3}"
+    ang_y="${PI/2}"
   />
   <xacro:tof_sensor
     tof_name="sr"
-    pos_x="${-chassis_x*0.2}"
-    pos_y="${-chassis_y*0.35}"
+    pos_x="${-0.0125}"
+    pos_y="${-0.145}"
     pos_z="0"
     ang_r="0"
     ang_p="0"
-    ang_y="${-2*PI/3}"
+    ang_y="${-PI/2}"
   />
   <xacro:tof_sensor
     tof_name="bm"
-    pos_x="${-chassis_x*0.4}"
+    pos_x="${-0.177}"
     pos_y="0"
     pos_z="0"
